File: kicad/crosstomp.sch (KiCad schematic (older format))
At the start: 43 parts, among them P1 IN, P2 9V, P3 HIGH, P4 SUM, P5 LOW, SW1 Phase, U1 TLE2426, U2 TLC274, U3 TL072

Commit message: 19/08/2014
Parts:
- C1, C2, C3, C6, C7, R1, R10, R11, R12, R13, R14, R15, R16, R17, R2, R3, R4, R5, R6, R7, R8, R9: footprint (none) -> SMD_Packages:SMD-0805
- C10, C4, C5, C8, C9: footprint (none) -> Capacitors_SMD:c_elec_5x5.3
- P1, P2: footprint (none) -> Pin_Headers:Pin_Header_Straight_1x02
- P3, P4, P5: footprint (none) -> Pin_Headers:Pin_Header_Straight_1x01
- RV1, RV2, RV5, RV6, RV7: footprint (none) -> Pin_Headers:Pin_Header_Straight_1x03
- RV3.1: renamed from RV3; footprint (none) -> Pin_Headers:Pin_Header_Straight_1x03
- RV3.2: renamed from RV4; footprint (none) -> Pin_Headers:Pin_Header_Straight_1x03
- SW1: footprint (none) -> Connect:SIL-9
- U1: footprint (none) -> Discret:TO92
- U2, U3: footprint (none) -> Housings_SOIC:SOIC-8_N
Other:
- moved on the sheet: C2, C3, C4, C5, R11, R12, R13, R9

Commit message: board design
Parts:
- removed C2, C3: 0.1 uF, SMD_Packages:SMD-0805, symbol C
- removed SW1: Phase, Connect:SIL-9, symbol SW-3PDT
- removed U1: TLE2426, Discret:TO92, symbol TLE2426
- added C2: 10 uF, Capacitors_SMD:c_elec_5x5.3, symbol CP1
- added SW1.1, SW1.2, SW1.3: SW-SPDT, Pin_Headers:Pin_Header_Straight_1x03, symbol SW-SPDT
- added U1: TLE2426-SOIC, Housings_SOIC:SOIC-8_N, symbol TLE2426-SOIC
- C5: value 10 uF -> 1 uF
- U2: footprint Housings_SOIC:SOIC-8_N -> SMD_Packages:SOIC-14_N
Connections:
- net GND: now also C2.1, SW1.1.2, U1.1 (VOUT); no longer C5.1
- net V+: now also U1.3 (VIN)
- net V-: now also C2.2, U1.2 (COM)
- net at C7.1, R4.2, U2.14: now also SW1.2.2
- net at R10.2, U3.1: now also SW1.3.1
- net at R13.1, R17.2: now also SW1.3.2
- net at R9.1: now also SW1.1.3, SW1.2.1
- new net: C5.1, U1.8 (NR)
- new net: SW1.2.3, SW1.3.3
Other:
- moved on the sheet: C4, C5, P2, U3A
