File: kicad/crosstomp.kicad_pcb (KiCad board)
At the start: 2 copper layers, 57.1 x 42.5 mm, 43 parts, among them P1 IN, P2 9V, P3 HIGH, P4 SUM, P5 LOW, SW1 Phase, U1 TLE2426, U2 TLC274, U3 TL072

Commit message: board design
Parts:
- removed C3: 0.1 uF, SMD_Packages:SMD-0805
- removed SW1: Phase, Connect:SIL-9
- added SW1.1: SW-SPDT, Pin_Headers:Pin_Header_Straight_1x03, F.Cu at (113.0, 83.8)
- added SW1.2: SW-SPDT, Pin_Headers:Pin_Header_Straight_1x03, F.Cu at (120.7, 83.8)
- added SW1.3: SW-SPDT, Pin_Headers:Pin_Header_Straight_1x03, F.Cu at (128.3, 83.8)
- C2: value 0.1 uF -> 10 uF; footprint SMD_Packages:SMD-0805 -> Capacitors_SMD:c_elec_5x5.3
- C5: value 10 uF -> 1 uF
- U1: value TLE2426 -> TLE2426-SOIC; footprint Discret:TO92 -> Housings_SOIC:SOIC-8_N
- U2: footprint Housings_SOIC:SOIC-8_N -> SMD_Packages:SOIC-14_N
- moved R5 77.0 mm to (168.2, 45.6)
- moved R3 62.1 mm to (158.3, 73.9)
- moved R2 61.2 mm to (154.1, 73.9)
- moved RV1 57.3 mm to (156.8, 62.9)
- moved R8 51.7 mm to (142.9, 89.9)
- moved C6 51.6 mm to (167.1, 57.3)
- moved R6 51.5 mm to (144.1, 85.9)
- moved R4 51.1 mm to (168.2, 43.1)
- moved RV2 46.5 mm to (147.6, 71.1)
- moved R13 42.3 mm to (130.8, 78.7), turned to 90 degrees
- moved P4 41.1 mm to (130.8, 59.1)
- moved C4 40.5 mm to (165.2, 63.5)
- moved R12 39.6 mm to (130.8, 74.7), turned to 270 degrees
- moved P5 38.4 mm to (130.8, 67.9)
- moved C5 35.4 mm to (83.8, 72.4), turned to 180 degrees
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Connections:
- C2 pad 2: V+ -> V-
- C5 pad 1: GND -> Net-(C5-Pad1)
- U1 pad 1: V+ -> GND
- U1 pad 3: GND -> V+
Routing:
- net GND: track 87.7 -> 47.5 mm, vias 3 -> 1
- net V-: track 31.5 -> 0.00 mm, vias 1 -> 0
- net Net-(C1-Pad1): track 26.0 -> 0.00 mm, vias 2 -> 0
- net Net-(R3-Pad1): track 24.7 -> 0.00 mm, vias 2 -> 0
- net Net-(R13-Pad1): track 2.98 -> 26.2 mm
- net V+: track 22.1 -> 0.00 mm
- net Net-(R2-Pad1): track 22.0 -> 0.00 mm, vias 2 -> 0
- net Net-(R8-Pad2): track 21.1 -> 0.00 mm, vias 1 -> 0
- net Net-(R4-Pad1): track 20.7 -> 0.00 mm, vias 1 -> 0
- net Net-(R12-Pad1): track 18.1 -> 3.33 mm
- net Net-(R11-Pad2): track 19.2 -> 6.56 mm, vias 2 -> 0
- net Net-(R3-Pad2): track 12.6 -> 0.00 mm, vias 2 -> 0
- net Net-(C10-Pad1): track 18.1 -> 6.07 mm, vias 2 -> 0
- net Net-(R10-Pad1): track 18.8 -> 7.65 mm, vias 2 -> 0
- net Net-(C6-Pad2): track 10.9 -> 0.00 mm, vias 1 -> 0
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Other:
- board size 57.1 x 42.5 mm -> 58.4 x 45.7 mm
- net class Default: via_dia 1.27 -> 1.016; via_drill 0.635 -> 0.508

Commit message: pcb routed and plots generated
Parts:
- moved C6 69.3 mm to (97.8, 55.2), turned to 180 degrees
- moved RV1 65.2 mm to (92.1, 55.2), turned to 90 degrees
- moved R3 60.9 mm to (97.8, 66.7), turned to 180 degrees
- moved R4 60.2 mm to (114.3, 69.8)
- moved C4 58.9 mm to (106.7, 70.5)
- moved RV2 56.2 mm to (92.1, 62.9), turned to 90 degrees
- moved R5 56.1 mm to (114.3, 61.0)
- moved P2 53.5 mm to (92.1, 82.5), turned to 90 degrees
- moved R6 51.2 mm to (97.8, 64.1), turned to 180 degrees
- moved R2 50.1 mm to (104.8, 65.4), turned to 180 degrees
- moved RV3.1 48.1 mm to (102.2, 47.0), turned to 180 degrees
- moved R8 47.4 mm to (114.3, 52.1), turned to 180 degrees
- moved C7 46.5 mm to (97.8, 61.6), turned to 180 degrees
- moved RV3.2 38.6 mm to (109.9, 47.0), turned to 180 degrees
- moved C2 15.4 mm to (106.7, 78.1), turned to 90 degrees
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Routing:
- net GND: track 47.5 -> 156.7 mm, vias 1 -> 2
- net V-: track 0.00 -> 78.2 mm, vias 0 -> 1
- net V+: track 0.00 -> 76.3 mm, vias 0 -> 1
- net Net-(C6-Pad1): track 0.00 -> 72.0 mm
- net Net-(R7-Pad2): track 0.00 -> 54.4 mm, vias 0 -> 1
- net Net-(C7-Pad1): track 0.00 -> 51.3 mm, vias 0 -> 2
- net Net-(R4-Pad1): track 0.00 -> 48.2 mm, vias 0 -> 1
- net Net-(R12-Pad1): track 3.33 -> 50.6 mm
- net Net-(C7-Pad2): track 0.00 -> 43.9 mm
- net Net-(R2-Pad2): track 0.00 -> 26.9 mm
- net Net-(C1-Pad1): track 0.00 -> 22.7 mm, vias 0 -> 3
- net Net-(R12-Pad2): track 2.16 -> 22.0 mm, vias 0 -> 2
- net Net-(R3-Pad1): track 0.00 -> 18.5 mm
- net Net-(C6-Pad2): track 0.00 -> 18.1 mm
- net Net-(R14-Pad2): track 4.90 -> 21.3 mm
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- added copper zone on B.Cu, net GND
Other:
- board size 58.4 x 45.7 mm -> 45.7 x 42.5 mm
- net class Default: via_dia 1.016 -> 0.762
- rule via_min_size: 0.889 -> 0.762
- board text added: "CrossStomp v1 www.dolganoff.com"
